Commit message: 최태오 커밋

File: Manipulator_study/arduinobot_description/urdf/arduinobot.urdf.xacro (robot description, xacro)
@@ -53,5 +53,5 @@
         <parent link="world"/>
         <child link="base_link"/>
-        <origin xyz="100 0 0" rpy="0 0 0"/>
+        <origin xyz="120 0 0" rpy="0 0 ${PI/2}"/>
     </joint>
     <!-- 위에 쓰고 CMake로-->
@@ -85,5 +85,5 @@
         <origin rpy="0 0 0" xyz="0 0 0"/><!-- T matrix, 즉 z축으로 0.307 만큼 올라가는 뜻! -->
         <!--조인트 움직임 한계 조절, effort는 토크 -->
-        <limit lower="${-PI}" upper="${PI}" effort="${effort}" velocity="${velocity}"/>
+        <limit lower="${-2*PI}" upper="${2*PI}" effort="${effort}" velocity="${velocity}"/>
         <!--xacro로 지정한 변수를 집어넣어서 유지보수를 쉽게!! ${변수}로 사용가능. 이때 연산은 안이든 밖이든 상관 없는 듯-->
         <!-- 90 이동 제한이라 PI/2-->
@@ -195,17 +195,17 @@
         <xacro:default_inertial mass="500.0"/>
         <visual>
-            <!-- <origin rpy="0 0 0" xyz="0 0 10"/> -->
-            <origin rpy="-${PI/2} 0 0" xyz="0 0 1"/>
-            <geometry>
-                <!-- <box size="10 1 10"/>  -->
-                <mesh filename="package://arduinobot_description/meshes/simplebox_box_v5.stl" scale="0.2 0.2 0.2"/>
-            </geometry>
-        </visual>
-        <collision>
-            <!-- <origin rpy="0 0 0" xyz="0 0 10"/> -->
-            <origin rpy="-${PI/2} 0 0" xyz="0 0 1"/>
-            <geometry>
-                <!-- <box size="10 1 10"/> -->
-                <mesh filename="package://arduinobot_description/meshes/simplebox_box_v5.stl" scale="0.2 0.2 0.2"/>
+            <origin rpy="0 0 0" xyz="0 0 10"/>
+            <!-- <origin rpy="-${PI/2} 0 0" xyz="0 0 15"/> -->
+            <geometry>
+                <box size="10 0.5 10"/>
+                <!-- <mesh filename="package://arduinobot_description/meshes/simplebox_box_v5.stl" scale="0.2 0.2 0.2"/>              -->
+            </geometry>
+        </visual>
+        <collision>
+            <origin rpy="0 0 0" xyz="0 0 10"/>
+            <!-- <origin rpy="-${PI/2} 0 0" xyz="0 0 15"/> -->
+            <geometry>
+                <box size="10 0.5 10"/>
+                <!-- <mesh filename="package://arduinobot_description/meshes/simplebox_box_v5.stl" scale="0.2 0.2 0.2"/>              -->
             </geometry>
             <!-- Add Gazebo friction parameters here -->

File: Manipulator_study/arduinobot_description/urdf/arduinobot_ros2_control.xacro (robot description, xacro)
@@ -14,6 +14,6 @@
             <command_interface name="position">
                 <!--파라미터, 최대 90, 최소 -90, 두배로 늘리기-->
-                <param name="max">${PI}</param>
-                <param name="min">-${PI}</param>
+                <param name="max">${2*PI}</param>
+                <param name="min">-${2*PI}</param>
             </command_interface>
             <!--하드웨어에서 명령 읽기-->

Commit message: 최태오 커밋

File: Manipulator_study/arduinobot_description/urdf/arduinobot.urdf.xacro (robot description, xacro)
@@ -53,5 +53,5 @@
         <parent link="world"/>
         <child link="base_link"/>
-        <origin xyz="120 0 0" rpy="0 0 ${PI/2}"/>
+        <origin xyz="119.97 0 0" rpy="0 0 ${PI/2}"/>
     </joint>
     <!-- 위에 쓰고 CMake로-->
@@ -214,4 +214,5 @@
                 <surface>
                     <contact>
+                        <!-- <collide_bitmask>0x02</collide_bitmask> -->
                         <ode>
                         <!-- <kp>100000.0</kp>
@@ -230,4 +231,19 @@
             </gazebo>
         </collision>
+        <visual>
+            <origin rpy="0 0 0" xyz="0 0 5"/>
+            <!-- <origin rpy="-${PI/2} 0 0" xyz="0 0 15"/> -->
+            <geometry>
+                <box size="10 1 0.5"/>
+                <!-- <mesh filename="package://arduinobot_description/meshes/simplebox_box_v5.stl" scale="0.2 0.2 0.2"/>              -->
+            </geometry>
+        </visual>
+        <collision>
+            <origin rpy="0 0 0" xyz="0 0 5"/>
+            <geometry>
+                <box size="10 1 0.5"/>
+                <!-- <mesh filename="package://arduinobot_description/meshes/simplebox_box_v5.stl" scale="0.2 0.2 0.2"/>              -->
+            </geometry>
+        </collision>
     </link>
     <joint name="joint_6" type="revolute">
